Commit message: Made PSMs more modular in preparation for reuse in simulation.
Added support for simulation modularity and control.

Made camera functional.

Minor changes to accomodate simulation.

Added simplified collisions.

File: model/PSM1.urdf.xacro (robot description, xacro)
@@ -1,11 +1,11 @@
 <?xml version="1.0" ?>
 <robot name="dvrk_psm" xmlns:xacro="http://www.ros.org/wiki/xacro">
-  <!-- Macros -->
-  <xacro:include filename="$(find cwru_davinci_geometry_models)/model/psm.urdf.xacro"/>
-  <link name="world"/>
-  <xacro:psm_sca
-      prefix="$(arg prefix)"
-      parent_link="world"
-      xyz="-0.25 0.0 0.5" rpy="0.0 0.0 3.1415926"
-      color="Green"/>
+	<!-- Macros -->
+	<xacro:include filename="$(find cwru_davinci_geometry_models)/model/PSM_generic.urdf.xacro"/>
+	<link name="world"/>
+	<xacro:psm_generic
+		prefix="PSM1"
+		xyz="-0.25 0.0 0.5" rpy="0.0 0.0 3.1415926"
+		color="Green"
+	/>
 </robot>

File: model/PSM2.urdf.xacro (robot description, xacro)
@@ -2,10 +2,10 @@
 <robot name="dvrk_psm" xmlns:xacro="http://www.ros.org/wiki/xacro">
   <!-- Macros -->
-  <xacro:include filename="$(find cwru_davinci_geometry_models)/model/psm.urdf.xacro"/>
+  <xacro:include filename="$(find cwru_davinci_geometry_models)/model/PSM_generic.urdf.xacro"/>
   <link name="world"/>
-  <xacro:psm_sca
-      prefix="$(arg prefix)"
-      parent_link="world"
+  <xacro:psm_generic
+      prefix="PSM2"
       xyz="0.25 0.0 0.5" rpy="0.0 0.0 -3.1415926"
-      color="Yellow"/>
+      color="Yellow"
+  />
 </robot>

File: model/PSM3.urdf.xacro (robot description, xacro)
@@ -1,10 +1,11 @@
 <?xml version="1.0" ?>
 <robot name="dvrk_psm" xmlns:xacro="http://www.ros.org/wiki/xacro">
-  <!-- Macros -->
-  <xacro:include filename="$(find cwru_davinci_geometry_models)/model/psm.urdf.xacro"/>
-  <link name="world"/>
-  <xacro:psm_caudier
-    prefix="$(arg prefix)"
-    parent_link="world"
-    xyz="0.50 0.0 0.5" rpy="0.0 0.0 -3.1415926"/>
+	<!-- Macros -->
+	<xacro:include filename="$(find cwru_davinci_geometry_models)/model/PSM_generic.urdf.xacro"/>
+	<link name="world"/>
+	<xacro:psm_generic
+		prefix="PSM3"
+		xyz="0.50 0.0 0.5" rpy="0.0 0.0 -3.1415926"
+		color="Red"
+	/>
 </robot>

File: model/camera.urdf.xacro (robot description, xacro)
@@ -2,6 +2,7 @@
 <robot name="dvrk_camera" xmlns:xacro="http://www.ros.org/wiki/xacro">
 	<!--TODO Sort out include properly-->
+	<link name="world"/>
 	<joint name="left_camera_joint" type="fixed">
-		<parent link="camera"/>
+		<parent link="world"/>
 		<child link="left_camera_link"/>
 		<origin rpy="0.0 1.5708 1.5708" xyz="0.005 0.00 0.5"/>
@@ -13,5 +14,4 @@
 				<box size="0.03 0.01 0.01"/>
 			</geometry>
-			<material name="red"/>
 		</visual>
 		<inertial>
@@ -22,5 +22,5 @@
 	</link>
 	<joint name="right_camera_joint" type="fixed">
-		<parent link="camera"/>
+		<parent link="world"/>
 		<child link="right_camera_link"/>
 		<origin rpy="0.0 1.5708 1.5708" xyz="-0.005 0.0 0.5"/>
@@ -32,5 +32,4 @@
 				<box size="0.03 0.01 0.01"/>
 			</geometry>
-			<material name="red"/>
 		</visual>
 		<inertial>
@@ -68,6 +67,6 @@
 				<alwaysOn>true</alwaysOn>
 				<updateRate>0.0</updateRate>
-				<cameraName>/davinci_endo/right</cameraName>
-				<imageTopicName>image_rect_color</imageTopicName>
+				<cameraName>/unsynced/right</cameraName>
+				<imageTopicName>image_raw</imageTopicName>
 				<cameraInfoTopicName>camera_info</cameraInfoTopicName>
 				<frameName>right_camera_link</frameName>
@@ -108,6 +107,6 @@
 				<alwaysOn>true</alwaysOn>
 				<updateRate>0.0</updateRate>
-				<cameraName>/davinci_endo/left</cameraName>
-				<imageTopicName>image_rect_color</imageTopicName>
+				<cameraName>/unsynced/left</cameraName>
+				<imageTopicName>image_raw</imageTopicName>
 				<cameraInfoTopicName>camera_info</cameraInfoTopicName>
 				<frameName>left_camera_optical_frame</frameName>

File: model/psm.base.urdf.xacro (robot description, xacro)
@@ -209,4 +209,10 @@
 				</geometry>
 			</visual>
+			<collision>
+				<origin rpy="0 0 0" xyz="0.005 0.18 -0.0025"/>
+				<geometry>
+					<box size="0.04 0.5 0.08"/>
+				</geometry>
+			</collision>
 			<inertial>
 				<origin xyz="0 0 0" rpy="0 0 0"/>
@@ -239,4 +245,16 @@
 				</geometry>
 			</visual>
+			<collision>
+				<origin rpy="0 0 0" xyz="0.005 0 -0.01"/>
+				<geometry>
+					<box size="0.045 0.07 0.09"/>
+				</geometry>
+			</collision>
+			<collision>
+				<origin rpy="0 0 0" xyz="0.00 0 0.2"/>
+				<geometry>
+					<box size="0.0075 0.0075 0.435"/>
+				</geometry>
+			</collision>
 			<inertial>
 				<origin xyz="0 0 0" rpy="0 0 0"/>
@@ -303,9 +321,8 @@
 		<transmission name="${prefix}tran1">
 			<type>transmission_interface/SimpleTransmission</type>
-			<joint name="${prefix}outer_yaw_joint">
-				<hardwareInterface>EffortJointInterface</hardwareInterface>
+			<joint name="outer_yaw">
+				<hardwareInterface>hardware_interface/EffortJointInterface</hardwareInterface>
 			</joint>
 			<actuator name="${prefix}motor1">
-				<hardwareInterface>EffortJointInterface</hardwareInterface>
 				<mechanicalReduction>1</mechanicalReduction>
 			</actuator>
@@ -313,69 +330,41 @@
 		<transmission name="${prefix}tran2">
 			<type>transmission_interface/SimpleTransmission</type>
-			<joint name="${prefix}outer_pitch_joint">
-				<hardwareInterface>EffortJointInterface</hardwareInterface>
+			<joint name="outer_pitch">
+				<hardwareInterface>hardware_interface/EffortJointInterface</hardwareInterface>
 			</joint>
 			<actuator name="${prefix}motor2">
-				<hardwareInterface>EffortJointInterface</hardwareInterface>
 				<mechanicalReduction>1</mechanicalReduction>
 			</actuator>
 		</transmission>
-		<transmission name="${prefix}tran2_1">
-			<type>transmission_interface/SimpleTransmission</type>
-			<joint name="${prefix}outer_pitch_joint_1">
-				<hardwareInterface>EffortJointInterface</hardwareInterface>
-			</joint>
-			<actuator name="${prefix}motor2_1">
-				<hardwareInterface>EffortJointInterface</hardwareInterface>
-				<mechanicalReduction>1</mechanicalReduction>
-			</actuator>
-		</transmission>
-		<transmission name="${prefix}tran2_2">
-			<type>transmission_interface/SimpleTransmission</type>
-			<joint name="${prefix}outer_pitch_joint_2">
-				<hardwareInterface>EffortJointInterface</hardwareInterface>
-			</joint>
-			<actuator name="${prefix}motor2_2">
-				<hardwareInterface>EffortJointInterface</hardwareInterface>
-				<mechanicalReduction>1</mechanicalReduction>
-			</actuator>
-		</transmission>
-		<transmission name="${prefix}tran2_3">
-			<type>transmission_interface/SimpleTransmission</type>
-			<joint name="${prefix}outer_pitch_joint_3">
-				<hardwareInterface>EffortJointInterface</hardwareInterface>
-			</joint>
-			<actuator name="${prefix}motor2_3">
-				<hardwareInterface>EffortJointInterface</hardwareInterface>
-				<mechanicalReduction>-1</mechanicalReduction>
-			</actuator>
-		</transmission>
-		<transmission name="${prefix}tran2_4">
-			<type>transmission_interface/SimpleTransmission</type>
-			<joint name="${prefix}outer_pitch_joint_4">
-				<hardwareInterface>EffortJointInterface</hardwareInterface>
-			</joint>
-			<actuator name="${prefix}motor2_4">
-				<hardwareInterface>EffortJointInterface</hardwareInterface>
-				<mechanicalReduction>-1</mechanicalReduction>
-			</actuator>
-		</transmission>
-		<transmission name="${prefix}tran2_5">
-			<type>transmission_interface/SimpleTransmission</type>
-			<joint name="${prefix}outer_pitch_joint_5">
-				<hardwareInterface>EffortJointInterface</hardwareInterface>
-			</joint>
-			<actuator name="${prefix}motor2_5">
-				<hardwareInterface>EffortJointInterface</hardwareInterface>
-				<mechanicalReduction>1</mechanicalReduction>
-			</actuator>
-		</transmission>
+		<gazebo>
+			<plugin name="mimic_1" filename="libroboticsgroup_gazebo_mimic_joint_plugin.so">
+				<joint>outer_pitch</joint>
+				<mimicJoint>outer_pitch_1</mimicJoint>
+			</plugin>
+			<plugin name="mimic_2" filename="libroboticsgroup_gazebo_mimic_joint_plugin.so">
+				<joint>outer_pitch</joint>
+				<mimicJoint>outer_pitch_2</mimicJoint>
+			</plugin>
+			<plugin name="mimic_3" filename="libroboticsgroup_gazebo_mimic_joint_plugin.so">
+				<joint>outer_pitch</joint>
+				<mimicJoint>outer_pitch_3</mimicJoint>
+				<multiplier>-1.0</multiplier>
+			</plugin>
+			<plugin name="mimic_4" filename="libroboticsgroup_gazebo_mimic_joint_plugin.so">
+				<joint>outer_pitch</joint>
+				<mimicJoint>outer_pitch_4</mimicJoint>
+				<multiplier>-1.0</multiplier>
+			</plugin>
+			<plugin name="mimic_5" filename="libroboticsgroup_gazebo_mimic_joint_plugin.so">
+				<joint>outer_pitch</joint>
+				<mimicJoint>outer_pitch_5</mimicJoint>
+			</plugin>
+		</gazebo>
 		<transmission name="${prefix}tran3">
 			<type>transmission_interface/SimpleTransmission</type>
-			<joint name="${prefix}outer_insertion_joint">
-				<hardwareInterface>EffortJointInterface</hardwareInterface>
+			<joint name="outer_insertion">
+				<hardwareInterface>hardware_interface/EffortJointInterface</hardwareInterface>
 			</joint>
 			<actuator name="${prefix}motor3">
-				<hardwareInterface>EffortJointInterface</hardwareInterface>
 				<mechanicalReduction>1</mechanicalReduction>
 			</actuator>
@@ -383,9 +372,8 @@
 		<transmission name="${prefix}tran4">
 			<type>transmission_interface/SimpleTransmission</type>
-			<joint name="${prefix}outer_roll_joint">
-				<hardwareInterface>EffortJointInterface</hardwareInterface>
+			<joint name="outer_roll">
+				<hardwareInterface>hardware_interface/EffortJointInterface</hardwareInterface>
 			</joint>
 			<actuator name="${prefix}motor4">
-				<hardwareInterface>EffortJointInterface</hardwareInterface>
 				<mechanicalReduction>1</mechanicalReduction>
 			</actuator>

File: model/psm.tool.sca.urdf.xacro (robot description, xacro)
@@ -7,6 +7,6 @@
 		<!-- joint 5: Outer wrist pitch joint -->
 		<joint name="outer_wrist_pitch" type="revolute">
-			<parent link="${prefix}tool_wrist_shaft_link"/>
-			<child link="${prefix}tool_wrist_sca_link"/>
+			<parent link="${prefix}_tool_wrist_shaft_link"/>
+			<child link="${prefix}_tool_wrist_sca_link"/>
 			<axis xyz="0 0 1"/>
 			<origin rpy="-1.5708 -1.5708 0" xyz="0 0 0"/>
@@ -14,5 +14,5 @@
 		</joint>
 		<!-- link 5: tool_wrist_sca_link -->
-		<link name="${prefix}tool_wrist_sca_link">
+		<link name="${prefix}_tool_wrist_sca_link">
 			<visual>
 				<origin rpy="1.5708 3.1416 0" xyz="0.0051 0.0032 0"/>
@@ -22,9 +22,7 @@
 			</visual>
 			<collision>
-				<origin rpy="1.5708 3.1416 0" xyz="0.0051 0.0032 0"/>
-				<geometry>
-					<!-- TODO: Switch to downpoly'd versions for collision detection-->
-					<mesh filename="package://cwru_davinci_geometry_models/meshes/psm/tool_wrist_sca_link.dae"/>
-					<!--box size="0 0 0" /-->
+				<origin rpy="1.5708 3.1416 0" xyz="0.0051 0 0"/>
+				<geometry>
+					<box size="0.011 0.007 0.005" />
 				</geometry>
 			</collision>
@@ -36,10 +34,10 @@
 			</inertial>
 		</link>
-		<gazebo reference="${prefix}tool_wrist_sca_link">
+		<gazebo reference="${prefix}_tool_wrist_sca_link">
 		</gazebo>
 		<!-- joint 6: Outer wrist yaw joint -->
 		<joint name="outer_wrist_yaw" type="revolute">
-			<parent link="${prefix}tool_wrist_sca_link"/>
-			<child link="${prefix}tool_wrist_sca_shaft_link"/>
+			<parent link="${prefix}_tool_wrist_sca_link"/>
+			<child link="${prefix}_tool_wrist_sca_shaft_link"/>
 			<axis xyz="0 0 1"/>
 			<origin rpy="-1.5708 -1.5708 0" xyz="0.0091 0 0"/>
@@ -48,5 +46,5 @@
 		</joint>
 		<!-- link 6: tool_wrist_sca_shaft_link -->
-		<link name="${prefix}tool_wrist_sca_shaft_link">
+		<link name="${prefix}_tool_wrist_sca_shaft_link">
 			<visual>
 				<origin rpy="0 0 0" xyz="0 -0.0002 -0.0025"/>
@@ -61,8 +59,8 @@
 			</inertial>
 		</link>
-		<!-- joint 7-0: Outer open angle 1	-->
+		<!-- joint 7-0: Outer open angle 1-->
 		<joint name="jaw" type="revolute">
-			<parent link="${prefix}tool_wrist_sca_shaft_link"/>
-			<child link="${prefix}tool_wrist_sca_ee_link_0"/>
+			<parent link="${prefix}_tool_wrist_sca_shaft_link"/>
+			<child link="${prefix}_tool_wrist_sca_ee_link_0"/>
 			<axis xyz="0 0 1"/>
 			<origin rpy="0 0 0" xyz="0 0 0"/>
@@ -70,16 +68,21 @@
 		</joint>
 		<!-- link 7-0: Outer open angle virtual -->
-		<link name="${prefix}tool_wrist_sca_ee_link_0">
-			<visual>
+		<link name="${prefix}_tool_wrist_sca_ee_link_0">
+			<!--visual>
 				<origin rpy="0 0 0" xyz="0 0 0"/>
 				<geometry>
-					<box size="0 0 0" />
-				</geometry>
-			</visual>
+					<box size="0.1 0.1 0.1" />
+				</geometry>
+			</visual-->
+			<inertial>
+				<origin xyz="0 0 0" rpy="0 0 0"/>
+				<mass value="0.05"/>
+				<inertia ixx="0.01" ixy="0.0" ixz="0.0" iyy="0.01" iyz="0.0" izz="0.005"/>
+			</inertial>
 		</link>
 		<!-- joint 7-1: Outer open angle 1	-->
 		<joint name="jaw_mimic_1" type="revolute">
-			<parent link="${prefix}tool_wrist_sca_shaft_link"/>
-			<child link="${prefix}tool_wrist_sca_ee_link_1"/>
+			<parent link="${prefix}_tool_wrist_sca_shaft_link"/>
+			<child link="${prefix}_tool_wrist_sca_ee_link_1"/>
 			<axis xyz="0 0 1"/>
 			<origin rpy="0 0 0" xyz="0 0 0"/>
@@ -88,5 +91,5 @@
 		</joint>
 		<!-- link 7-1: Outer open angle link 1 -->
-		<link name="${prefix}tool_wrist_sca_ee_link_1">
+		<link name="${prefix}_tool_wrist_sca_ee_link_1">
 			<visual>
 				<origin rpy="0 0 0" xyz="0 0 0"/>
@@ -103,6 +106,6 @@
 		<!-- joint 7-2: Outer open angle 2	 -->
 		<joint name="jaw_mimic_2" type="revolute">
-			<parent link="${prefix}tool_wrist_sca_shaft_link"/>
-			<child link="${prefix}tool_wrist_sca_ee_link_2"/>
+			<parent link="${prefix}_tool_wrist_sca_shaft_link"/>
+			<child link="${prefix}_tool_wrist_sca_ee_link_2"/>
 			<axis xyz="0 0 1"/>
 			<origin rpy="0 0 0" xyz="0 0 0"/>
@@ -111,5 +114,5 @@
 		</joint>
 		<!-- link 7-2: Outer open angle link 2 -->
-		<link name="${prefix}tool_wrist_sca_ee_link_2">
+		<link name="${prefix}_tool_wrist_sca_ee_link_2">
 			<visual>
 				<origin rpy="0 3.1516 0" xyz="0 0 0"/>
@@ -124,11 +127,5 @@
 			</inertial>
 		</link>
-		<!-- tool tip -->
-		<joint name="tool_tip" type="fixed">
-			<parent link="${prefix}tool_wrist_sca_shaft_link"/>
-			<child link="${prefix}tool_tip_link"/>
-			<origin rpy="0 ${PI/2} ${PI/2}" xyz="0 0.0102 0"/>
-		</joint>
-		<link name="${prefix}fingertip2">
+		<link name="${prefix}_fingertip2">
 			<visual>
 				<origin rpy="0 0 0" xyz="0.001 0.005 0.0005"/>
@@ -166,12 +163,12 @@
 		</link>
 		<!-- attach fingertip pad  -->
-		<joint name="${prefix}fingertip2_joint" type="fixed">
-			<parent link="${prefix}tool_wrist_sca_ee_link_2"/>
-			<child link="${prefix}fingertip2"/>
+		<joint name="${prefix}_fingertip2_joint" type="fixed">
+			<parent link="${prefix}_tool_wrist_sca_ee_link_2"/>
+			<child link="${prefix}_fingertip2"/>
 			<axis xyz="0 0 1"/>
 			<origin rpy="0 0 0" xyz="0 0 0"/>
 		</joint>
 		<!-- wsn: other fingertip -->
-		<link name="${prefix}fingertip1">
+		<link name="${prefix}_fingertip1">
 			<visual>
 				<origin rpy="0 0 0" xyz="-0.001 0.005 0.0005"/>
@@ -180,5 +177,5 @@
 				</geometry>
 			</visual>
-			<collision name="${prefix}fingertip1_collision">
+			<collision name="${prefix}_fingertip1_collision">
 				<origin rpy="0 0 0" xyz="-0.001 0.005 0.0005"/>
 				<geometry>
@@ -209,17 +206,17 @@
 		</link>
 		<!-- attach fingertip pad 1  -->
-		<joint name="${prefix}fingertip1_joint" type="fixed">
-			<parent link="${prefix}tool_wrist_sca_ee_link_1"/>
-			<child link="${prefix}fingertip1"/>
+		<joint name="${prefix}_fingertip1_joint" type="fixed">
+			<parent link="${prefix}_tool_wrist_sca_ee_link_1"/>
+			<child link="${prefix}_fingertip1"/>
 			<axis xyz="0 0 1"/>
 			<origin rpy="0 0 0" xyz="0 0 0"/>
 		</joint>
 		<!-- tool tip -->
-		<joint name="${prefix}tool_tip_joint_" type="fixed">
-			<parent link="${prefix}tool_wrist_sca_shaft_link"/>
-			<child link="${prefix}tool_tip_link"/>
+		<joint name="${prefix}_tool_tip_joint_" type="fixed">
+			<parent link="${prefix}_tool_wrist_sca_shaft_link"/>
+			<child link="${prefix}_tool_tip_link"/>
 			<origin rpy="0 ${PI/2} ${PI/2}" xyz="0 0.0102 0"/>
 		</joint>
-		<link name="${prefix}tool_tip_link">
+		<link name="${prefix}_tool_tip_link">
 			<visual>
 				<geometry>
@@ -230,58 +227,57 @@
 		</link>
 		<!--this colors the tool-tip fiducial red; oddly, this shows up in the camera view, but NOT in the rviz view -->
-		<gazebo reference="${prefix}tool_tip_link">
+		<gazebo reference="${prefix}_tool_tip_link">
 			<material>Gazebo/Red</material>
 		</gazebo>
 		<!--Color the sticky fingertips pink, for visibility-->
-		<gazebo reference="${prefix}fingertip1">
+		<gazebo reference="${prefix}_fingertip1">
 			<material>Gazebo/Purple</material>
 		</gazebo>
 		<!--Create the sticky fingertip.-->
 		<gazebo>
-			<plugin name="${prefix}fingertip1_finger" filename="libsticky_fingers.so">
+			<plugin name="${prefix}_fingertip1_finger" filename="libsticky_fingers.so">
 				<capacity>25</capacity>
-				<link>davinci::${prefix}tool_wrist_sca_ee_link_1</link>
+				<link>davinci_${prefix}::${prefix}_tool_wrist_sca_ee_link_1</link>
 			</plugin>
          	</gazebo>
-		<transmission name="${prefix}tran5">
+		<transmission name="${prefix}_tran5">
 			<type>transmission_interface/SimpleTransmission</type>
-			<joint name="${prefix}outer_wrist_pitch_joint">
-				<hardwareInterface>EffortJointInterface</hardwareInterface>
+			<joint name="outer_wrist_pitch">
+				<hardwareInterface>hardware_interface/EffortJointInterface</hardwareInterface>
 			</joint>
-			<actuator name="${prefix}motor5">
-				<hardwareInterface>EffortJointInterface</hardwareInterface>
+			<actuator name="${prefix}_motor5">
 				<mechanicalReduction>1</mechanicalReduction>
 			</actuator>
 		</transmission>
-		<transmission name="${prefix}tran6">
+		<transmission name="${prefix}_tran6">
 			<type>transmission_interface/SimpleTransmission</type>
-			<joint name="${prefix}outer_wrist_yaw_joint">
-				<hardwareInterface>EffortJointInterface</hardwareInterface>
+			<joint name="outer_wrist_yaw">
+				<hardwareInterface>hardware_interface/EffortJointInterface</hardwareInterface>
 			</joint>
-			<actuator name="${prefix}motor6">
-				<hardwareInterface>EffortJointInterface</hardwareInterface>
+			<actuator name="${prefix}_motor6">
 				<mechanicalReduction>1</mechanicalReduction>
 			</actuator>
 		</transmission>
-		<transmission name="${prefix}tran7">
+		<transmission name="${prefix}_tran7">
 			<type>transmission_interface/SimpleTransmission</type>
-			<joint name="${prefix}outer_wrist_open_angle_joint">
-				<hardwareInterface>EffortJointInterface</hardwareInterface>
+			<joint name="jaw">
+				<hardwareInterface>hardware_interface/EffortJointInterface</hardwareInterface>
 			</joint>
-			<actuator name="${prefix}motor7">
-				<hardwareInterface>EffortJointInterface</hardwareInterface>
+			<actuator name="${prefix}_motor7">
 				<mechanicalReduction>1</mechanicalReduction>
 			</actuator>
 		</transmission>
-		<transmission name="${prefix}tran7_mimic">
-			<type>transmission_interface/SimpleTransmission</type>
-			<joint name="${prefix}outer_wrist_open_angle_joint_mimic">
-				<hardwareInterface>EffortJointInterface</hardwareInterface>
-			</joint>
-			<actuator name="${prefix}motor7_mimic">
-				<hardwareInterface>EffortJointInterface</hardwareInterface>
-				<mechanicalReduction>1</mechanicalReduction>
-			</actuator>
-		</transmission>
+		<gazebo>
+			<plugin name="mimic_6" filename="libroboticsgroup_gazebo_mimic_joint_plugin.so">
+				<joint>jaw</joint>
+				<mimicJoint>jaw_mimic_1</mimicJoint>
+				<multiplier>0.5</multiplier>
+			</plugin>
+			<plugin name="mimic_7" filename="libroboticsgroup_gazebo_mimic_joint_plugin.so">
+				<joint>jaw</joint>
+				<mimicJoint>jaw_mimic_2</mimicJoint>
+				<multiplier>-0.5</multiplier>
+			</plugin>
+		</gazebo>
 	</xacro:macro>
 </robot>

File: model/psm.urdf.xacro (robot description, xacro)
@@ -8,5 +8,5 @@
   <xacro:macro name="psm_sca" params="prefix parent_link xyz rpy color">
     <xacro:psm
-        prefix="${prefix}"
+        prefix="${prefix}_"
         parent_link="${parent_link}"
         xyz="${xyz}" rpy="${rpy}"
@@ -18,10 +18,10 @@
   <xacro:macro name="psm_caudier" params="prefix parent_link xyz rpy color">
     <xacro:psm
-        prefix="${prefix}"
+        prefix="${prefix}_"
         parent_link="${parent_link}"
         xyz="${xyz}" rpy="${rpy}"
         color="${color}"/>
     <xacro:psm_tool_caudier
-        prefix="${prefix}"/>
+        prefix="${prefix}_"/>
   </xacro:macro>
 </robot>
