Commit message: Added dot board prop.
Got camera spawning properly.

Fixed baseline.

Fixed duplicate joint on tool tip.

Updated StickyFinger compat to remove crash.

Simplified PSM configuration and spawning.

Controller compatibility fixup.

Increased velocity limits for faster movement.

Made fiducial trackable in Gazebo.

File: model/PSM1.urdf.xacro (robot description, xacro)
@@ -5,7 +5,14 @@
   <link name="world"/>
   <xacro:psm_sca
-      prefix="$(arg prefix)"
+      prefix="PSM1"
       parent_link="world"
       xyz="-0.25 0.0 0.5" rpy="0.0 0.0 3.1415926"
       color="Green"/>
+  <!-- ros_control plugin -->
+	<gazebo>
+		<plugin name="gazebo_ros_control" filename="libgazebo_ros_control.so">
+			<robotNamespace>/dvrk/PSM1</robotNamespace>
+			<robotSimType>gazebo_ros_control/DefaultRobotHWSim</robotSimType>
+		</plugin>
+	</gazebo>
 </robot>

File: model/PSM2.urdf.xacro (robot description, xacro)
@@ -5,7 +5,14 @@
   <link name="world"/>
   <xacro:psm_sca
-      prefix="$(arg prefix)"
+      prefix="PSM2"
       parent_link="world"
       xyz="0.25 0.0 0.5" rpy="0.0 0.0 -3.1415926"
       color="Yellow"/>
+  <!-- ros_control plugin -->
+	<gazebo>
+		<plugin name="gazebo_ros_control" filename="libgazebo_ros_control.so">
+			<robotNamespace>/dvrk/PSM2</robotNamespace>
+			<robotSimType>gazebo_ros_control/DefaultRobotHWSim</robotSimType>
+		</plugin>
+	</gazebo>
 </robot>

File: model/camera.urdf.xacro (robot description, xacro)
@@ -2,6 +2,7 @@
 <robot name="dvrk_camera" xmlns:xacro="http://www.ros.org/wiki/xacro">
 	<!--TODO Sort out include properly-->
+	<link name="base"/>
 	<joint name="left_camera_joint" type="fixed">
-		<parent link="camera"/>
+		<parent link="base"/>
 		<child link="left_camera_link"/>
 		<origin rpy="0.0 1.5708 1.5708" xyz="0.005 0.00 0.5"/>
@@ -9,5 +10,5 @@
 	<link name="left_camera_link">
 		<visual>
-			<origin xyz="0 0 0.0" rpy="0 0 0"/>
+			<origin xyz="0 0 0.02" rpy="0 0 0"/>
 			<geometry>
 				<box size="0.03 0.01 0.01"/>
@@ -22,5 +23,5 @@
 	</link>
 	<joint name="right_camera_joint" type="fixed">
-		<parent link="camera"/>
+		<parent link="base"/>
 		<child link="right_camera_link"/>
 		<origin rpy="0.0 1.5708 1.5708" xyz="-0.005 0.0 0.5"/>
@@ -28,5 +29,5 @@
 	<link name="right_camera_link">
 		<visual>
-			<origin xyz="0 0 0.0" rpy="0 0 0"/>
+			<origin xyz="0 0 0.02" rpy="0 0 0"/>
 			<geometry>
 				<box size="0.03 0.01 0.01"/>
@@ -68,9 +69,9 @@
 				<alwaysOn>true</alwaysOn>
 				<updateRate>0.0</updateRate>
-				<cameraName>/davinci_endo/right</cameraName>
+				<cameraName>/right</cameraName>
 				<imageTopicName>image_rect_color</imageTopicName>
 				<cameraInfoTopicName>camera_info</cameraInfoTopicName>
 				<frameName>right_camera_link</frameName>
-				<hackBaseline>0.0</hackBaseline>
+				<hackBaseline>0.01</hackBaseline>
 				<distortionK1>0.0</distortionK1>
 				<distortionK2>0.0</distortionK2>
@@ -108,5 +109,5 @@
 				<alwaysOn>true</alwaysOn>
 				<updateRate>0.0</updateRate>
-				<cameraName>/davinci_endo/left</cameraName>
+				<cameraName>/left</cameraName>
 				<imageTopicName>image_rect_color</imageTopicName>
 				<cameraInfoTopicName>camera_info</cameraInfoTopicName>

File: model/psm.base.urdf.xacro (robot description, xacro)
@@ -6,5 +6,5 @@
 	<xacro:macro name="psm" params="prefix parent_link xyz rpy color">
 		<!-- fixed joint -->
-		<joint name="${prefix}fixed_joint" type="fixed">
+		<joint name="${prefix}_fixed_joint" type="fixed">
 			<parent link="${parent_link}"/>
 			<child link="${prefix}psm_base_link"/>
@@ -303,9 +303,8 @@
 		<transmission name="${prefix}tran1">
 			<type>transmission_interface/SimpleTransmission</type>
-			<joint name="${prefix}outer_yaw_joint">
-				<hardwareInterface>EffortJointInterface</hardwareInterface>
+			<joint name="outer_yaw">
+				<hardwareInterface>hardware_interface/EffortJointInterface</hardwareInterface>
 			</joint>
 			<actuator name="${prefix}motor1">
-				<hardwareInterface>EffortJointInterface</hardwareInterface>
 				<mechanicalReduction>1</mechanicalReduction>
 			</actuator>
@@ -313,69 +312,41 @@
 		<transmission name="${prefix}tran2">
 			<type>transmission_interface/SimpleTransmission</type>
-			<joint name="${prefix}outer_pitch_joint">
-				<hardwareInterface>EffortJointInterface</hardwareInterface>
+			<joint name="outer_pitch">
+				<hardwareInterface>hardware_interface/EffortJointInterface</hardwareInterface>
 			</joint>
 			<actuator name="${prefix}motor2">
-				<hardwareInterface>EffortJointInterface</hardwareInterface>
 				<mechanicalReduction>1</mechanicalReduction>
 			</actuator>
 		</transmission>
-		<transmission name="${prefix}tran2_1">
-			<type>transmission_interface/SimpleTransmission</type>
-			<joint name="${prefix}outer_pitch_joint_1">
-				<hardwareInterface>EffortJointInterface</hardwareInterface>
-			</joint>
-			<actuator name="${prefix}motor2_1">
-				<hardwareInterface>EffortJointInterface</hardwareInterface>
-				<mechanicalReduction>1</mechanicalReduction>
-			</actuator>
-		</transmission>
-		<transmission name="${prefix}tran2_2">
-			<type>transmission_interface/SimpleTransmission</type>
-			<joint name="${prefix}outer_pitch_joint_2">
-				<hardwareInterface>EffortJointInterface</hardwareInterface>
-			</joint>
-			<actuator name="${prefix}motor2_2">
-				<hardwareInterface>EffortJointInterface</hardwareInterface>
-				<mechanicalReduction>1</mechanicalReduction>
-			</actuator>
-		</transmission>
-		<transmission name="${prefix}tran2_3">
-			<type>transmission_interface/SimpleTransmission</type>
-			<joint name="${prefix}outer_pitch_joint_3">
-				<hardwareInterface>EffortJointInterface</hardwareInterface>
-			</joint>
-			<actuator name="${prefix}motor2_3">
-				<hardwareInterface>EffortJointInterface</hardwareInterface>
-				<mechanicalReduction>-1</mechanicalReduction>
-			</actuator>
-		</transmission>
-		<transmission name="${prefix}tran2_4">
-			<type>transmission_interface/SimpleTransmission</type>
-			<joint name="${prefix}outer_pitch_joint_4">
-				<hardwareInterface>EffortJointInterface</hardwareInterface>
-			</joint>
-			<actuator name="${prefix}motor2_4">
-				<hardwareInterface>EffortJointInterface</hardwareInterface>
-				<mechanicalReduction>-1</mechanicalReduction>
-			</actuator>
-		</transmission>
-		<transmission name="${prefix}tran2_5">
-			<type>transmission_interface/SimpleTransmission</type>
-			<joint name="${prefix}outer_pitch_joint_5">
-				<hardwareInterface>EffortJointInterface</hardwareInterface>
-			</joint>
-			<actuator name="${prefix}motor2_5">
-				<hardwareInterface>EffortJointInterface</hardwareInterface>
-				<mechanicalReduction>1</mechanicalReduction>
-			</actuator>
-		</transmission>
+		<gazebo>
+			<plugin name="mimic_1" filename="libroboticsgroup_gazebo_mimic_joint_plugin.so">
+				<joint>outer_pitch</joint>
+				<mimicJoint>outer_pitch_1</mimicJoint>
+			</plugin>
+			<plugin name="mimic_2" filename="libroboticsgroup_gazebo_mimic_joint_plugin.so">
+				<joint>outer_pitch</joint>
+				<mimicJoint>outer_pitch_2</mimicJoint>
+			</plugin>
+			<plugin name="mimic_3" filename="libroboticsgroup_gazebo_mimic_joint_plugin.so">
+				<joint>outer_pitch</joint>
+				<mimicJoint>outer_pitch_3</mimicJoint>
+				<multiplier>-1.0</multiplier>
+			</plugin>
+			<plugin name="mimic_4" filename="libroboticsgroup_gazebo_mimic_joint_plugin.so">
+				<joint>outer_pitch</joint>
+				<mimicJoint>outer_pitch_4</mimicJoint>
+				<multiplier>-1.0</multiplier>
+			</plugin>
+			<plugin name="mimic_5" filename="libroboticsgroup_gazebo_mimic_joint_plugin.so">
+				<joint>outer_pitch</joint>
+				<mimicJoint>outer_pitch_5</mimicJoint>
+			</plugin>
+		</gazebo>
 		<transmission name="${prefix}tran3">
 			<type>transmission_interface/SimpleTransmission</type>
-			<joint name="${prefix}outer_insertion_joint">
-				<hardwareInterface>EffortJointInterface</hardwareInterface>
+			<joint name="outer_insertion">
+				<hardwareInterface>hardware_interface/EffortJointInterface</hardwareInterface>
 			</joint>
 			<actuator name="${prefix}motor3">
-				<hardwareInterface>EffortJointInterface</hardwareInterface>
 				<mechanicalReduction>1</mechanicalReduction>
 			</actuator>
@@ -383,9 +354,8 @@
 		<transmission name="${prefix}tran4">
 			<type>transmission_interface/SimpleTransmission</type>
-			<joint name="${prefix}outer_roll_joint">
-				<hardwareInterface>EffortJointInterface</hardwareInterface>
+			<joint name="outer_roll">
+				<hardwareInterface>hardware_interface/EffortJointInterface</hardwareInterface>
 			</joint>
 			<actuator name="${prefix}motor4">
-				<hardwareInterface>EffortJointInterface</hardwareInterface>
 				<mechanicalReduction>1</mechanicalReduction>
 			</actuator>

File: model/psm.tool.sca.urdf.xacro (robot description, xacro)
@@ -11,5 +11,5 @@
 			<axis xyz="0 0 1"/>
 			<origin rpy="-1.5708 -1.5708 0" xyz="0 0 0"/>
-			<limit lower="-1.5707" upper="1.5707" velocity=".4" effort="1000"/>
+			<limit lower="-1.5707" upper="1.5707" velocity="20" effort="1000"/>
 		</joint>
 		<!-- link 5: tool_wrist_sca_link -->
@@ -45,5 +45,5 @@
 			<origin rpy="-1.5708 -1.5708 0" xyz="0.0091 0 0"/>
 			<!-- +/- 80 deg -->
-			<limit lower="-1.3963" upper="1.3963" velocity=".4" effort="1000"/>
+			<limit lower="-1.3963" upper="1.3963" velocity="10" effort="1000"/>
 		</joint>
 		<!-- link 6: tool_wrist_sca_shaft_link -->
@@ -67,14 +67,19 @@
 			<axis xyz="0 0 1"/>
 			<origin rpy="0 0 0" xyz="0 0 0"/>
-			<limit lower="0" upper="1.5707" velocity=".4" effort="1000"/>
+			<limit lower="0" upper="1.5707" velocity="10" effort="1000"/>
 		</joint>
 		<!-- link 7-0: Outer open angle virtual -->
 		<link name="${prefix}tool_wrist_sca_ee_link_0">
-			<visual>
+			<!--visual>
 				<origin rpy="0 0 0" xyz="0 0 0"/>
 				<geometry>
 					<box size="0 0 0" />
 				</geometry>
-			</visual>
+			</visual-->
+			<inertial>
+				<origin xyz="0 0 0" rpy="0 0 0"/>
+				<mass value="0.05"/>
+				<inertia ixx="0.01" ixy="0.0" ixz="0.0" iyy="0.01" iyz="0.0" izz="0.005"/>
+			</inertial>
 		</link>
 		<!-- joint 7-1: Outer open angle 1	-->
@@ -84,5 +89,5 @@
 			<axis xyz="0 0 1"/>
 			<origin rpy="0 0 0" xyz="0 0 0"/>
-			<limit lower="-1.5707" upper="1.5707" velocity=".4" effort="1000"/>
+			<limit lower="-1.5707" upper="1.5707" velocity="10" effort="1000"/>
 			<mimic joint="jaw" multiplier="0.5"/>
 		</joint>
@@ -107,5 +112,5 @@
 			<axis xyz="0 0 1"/>
 			<origin rpy="0 0 0" xyz="0 0 0"/>
-			<limit lower="-1.5707" upper="1.5707" velocity=".4" effort="1000"/>
+			<limit lower="-1.5707" upper="1.5707" velocity="10" effort="1000"/>
 			<mimic joint="jaw" multiplier="-0.5"/>
 		</joint>
@@ -125,9 +130,9 @@
 		</link>
 		<!-- tool tip -->
-		<joint name="tool_tip" type="fixed">
+		<!--joint name="tool_tip" type="fixed">
 			<parent link="${prefix}tool_wrist_sca_shaft_link"/>
 			<child link="${prefix}tool_tip_link"/>
 			<origin rpy="0 ${PI/2} ${PI/2}" xyz="0 0.0102 0"/>
-		</joint>
+		</joint-->
 		<link name="${prefix}fingertip2">
 			<visual>
@@ -216,8 +221,11 @@
 		</joint>
 		<!-- tool tip -->
-		<joint name="${prefix}tool_tip_joint_" type="fixed">
+		<!-- joint needs to be revolute (albeit immobile) to prevent Gazebo from optimizing the fiducial's position out.-->
+		<joint name="${prefix}tool_tip_joint_" type="revolute">
 			<parent link="${prefix}tool_wrist_sca_shaft_link"/>
 			<child link="${prefix}tool_tip_link"/>
 			<origin rpy="0 ${PI/2} ${PI/2}" xyz="0 0.0102 0"/>
+			<axis xyz="0 0 1"/>
+			<limit lower="-0.00001" upper="0.0001" velocity="10" effort="1000"/>
 		</joint>
 		<link name="${prefix}tool_tip_link">
@@ -228,4 +236,10 @@
 				</geometry>
 			</visual>
+			<!--Needs a dummy inertia value to link with the joint up above.-->
+			<inertial>
+				<origin xyz="0 0 0" rpy="0 0 0"/>
+				<mass value="0.1"/>
+				<inertia ixx="0.00" ixy="0.0" ixz="0.0" iyy="0.00" iyz="0.0" izz="0.000"/>
+			</inertial>
 		</link>
 		<!--this colors the tool-tip fiducial red; oddly, this shows up in the camera view, but NOT in the rviz view -->
@@ -241,47 +255,46 @@
 			<plugin name="${prefix}fingertip1_finger" filename="libsticky_fingers.so">
 				<capacity>25</capacity>
-				<link>davinci::${prefix}tool_wrist_sca_ee_link_1</link>
+				<link>davinci_${prefix}::${prefix}tool_wrist_sca_ee_link_1</link>
 			</plugin>
          	</gazebo>
-		<transmission name="${prefix}tran5">
+		<transmission name="${prefix}_tran5">
 			<type>transmission_interface/SimpleTransmission</type>
-			<joint name="${prefix}outer_wrist_pitch_joint">
-				<hardwareInterface>EffortJointInterface</hardwareInterface>
+			<joint name="outer_wrist_pitch">
+				<hardwareInterface>hardware_interface/EffortJointInterface</hardwareInterface>
 			</joint>
-			<actuator name="${prefix}motor5">
-				<hardwareInterface>EffortJointInterface</hardwareInterface>
+			<actuator name="${prefix}_motor5">
 				<mechanicalReduction>1</mechanicalReduction>
 			</actuator>
 		</transmission>
-		<transmission name="${prefix}tran6">
+		<transmission name="${prefix}_tran6">
 			<type>transmission_interface/SimpleTransmission</type>
-			<joint name="${prefix}outer_wrist_yaw_joint">
-				<hardwareInterface>EffortJointInterface</hardwareInterface>
+			<joint name="outer_wrist_yaw">
+				<hardwareInterface>hardware_interface/EffortJointInterface</hardwareInterface>
 			</joint>
-			<actuator name="${prefix}motor6">
-				<hardwareInterface>EffortJointInterface</hardwareInterface>
+			<actuator name="${prefix}_motor6">
 				<mechanicalReduction>1</mechanicalReduction>
 			</actuator>
 		</transmission>
-		<transmission name="${prefix}tran7">
+		<transmission name="${prefix}_tran7">
 			<type>transmission_interface/SimpleTransmission</type>
-			<joint name="${prefix}outer_wrist_open_angle_joint">
-				<hardwareInterface>EffortJointInterface</hardwareInterface>
+			<joint name="jaw">
+				<hardwareInterface>hardware_interface/EffortJointInterface</hardwareInterface>
 			</joint>
-			<actuator name="${prefix}motor7">
-				<hardwareInterface>EffortJointInterface</hardwareInterface>
+			<actuator name="${prefix}_motor7">
 				<mechanicalReduction>1</mechanicalReduction>
 			</actuator>
 		</transmission>
-		<transmission name="${prefix}tran7_mimic">
-			<type>transmission_interface/SimpleTransmission</type>
-			<joint name="${prefix}outer_wrist_open_angle_joint_mimic">
-				<hardwareInterface>EffortJointInterface</hardwareInterface>
-			</joint>
-			<actuator name="${prefix}motor7_mimic">
-				<hardwareInterface>EffortJointInterface</hardwareInterface>
-				<mechanicalReduction>1</mechanicalReduction>
-			</actuator>
-		</transmission>
+		<gazebo>
+			<plugin name="mimic_6" filename="libroboticsgroup_gazebo_mimic_joint_plugin.so">
+				<joint>jaw</joint>
+				<mimicJoint>jaw_mimic_1</mimicJoint>
+				<multiplier>0.5</multiplier>
+			</plugin>
+			<plugin name="mimic_7" filename="libroboticsgroup_gazebo_mimic_joint_plugin.so">
+				<joint>jaw</joint>
+				<mimicJoint>jaw_mimic_2</mimicJoint>
+				<multiplier>-0.5</multiplier>
+			</plugin>
+		</gazebo>
 	</xacro:macro>
 </robot>

Commit message: Removed powered joint in PSM tip for MoveIt integration.

File: model/PSM1.urdf.xacro (robot description, xacro)
@@ -8,6 +8,7 @@
       parent_link="world"
       xyz="-0.25 0.0 0.5" rpy="0.0 0.0 3.1415926"
-      color="Green"/>
-  <!-- ros_control plugin -->
+      color="Green"
+/>
+	<!-- ros_control plugin -->
 	<gazebo>
 		<plugin name="gazebo_ros_control" filename="libgazebo_ros_control.so">

File: model/psm.tool.sca.urdf.xacro (robot description, xacro)
@@ -129,10 +129,4 @@
 			</inertial>
 		</link>
-		<!-- tool tip -->
-		<!--joint name="tool_tip" type="fixed">
-			<parent link="${prefix}tool_wrist_sca_shaft_link"/>
-			<child link="${prefix}tool_tip_link"/>
-			<origin rpy="0 ${PI/2} ${PI/2}" xyz="0 0.0102 0"/>
-		</joint-->
 		<link name="${prefix}fingertip2">
 			<visual>
@@ -222,10 +216,8 @@
 		<!-- tool tip -->
 		<!-- joint needs to be revolute (albeit immobile) to prevent Gazebo from optimizing the fiducial's position out.-->
-		<joint name="${prefix}tool_tip_joint_" type="revolute">
+		<joint name="${prefix}tool_tip_joint_" type="fixed">
 			<parent link="${prefix}tool_wrist_sca_shaft_link"/>
 			<child link="${prefix}tool_tip_link"/>
 			<origin rpy="0 ${PI/2} ${PI/2}" xyz="0 0.0102 0"/>
-			<axis xyz="0 0 1"/>
-			<limit lower="-0.00001" upper="0.0001" velocity="10" effort="1000"/>
 		</joint>
 		<link name="${prefix}tool_tip_link">
@@ -239,5 +231,5 @@
 			<inertial>
 				<origin xyz="0 0 0" rpy="0 0 0"/>
-				<mass value="0.1"/>
+				<mass value="0.00001"/>
 				<inertia ixx="0.00" ixy="0.0" ixz="0.0" iyy="0.00" iyz="0.0" izz="0.000"/>
 			</inertial>
