Commit message: Modified psm.base.urdf.xacro and psm.tool.sca.urdf.xacro files with prefix joint names.

File: model/PSM1.urdf.xacro (robot description, xacro)
@@ -10,10 +10,10 @@
       color="Green"
 />
-	<!-- ros_control plugin -->
-	<gazebo>
-		<plugin name="gazebo_ros_control" filename="libgazebo_ros_control.so">
-			<robotNamespace>/dvrk/PSM1</robotNamespace>
-			<robotSimType>gazebo_ros_control/DefaultRobotHWSim</robotSimType>
-		</plugin>
-	</gazebo>
+    <!-- ros_control plugin -->
+    <gazebo>
+        <plugin name="gazebo_ros_control" filename="libgazebo_ros_control.so">
+            <robotNamespace>/dvrk/PSM1</robotNamespace>
+            <robotSimType>gazebo_ros_control/DefaultRobotHWSim</robotSimType>
+        </plugin>
+    </gazebo>
 </robot>

File: model/both_psms.urdf.xacro (robot description, xacro)
@@ -2,34 +2,32 @@
 <robot name="dvrk_psm" xmlns:xacro="http://www.ros.org/wiki/xacro">
 <!-- Macros -->
-<xacro:include filename="$(find cwru_davinci_geometry_models)/model/psm.urdf.xacro"/>
-	<link name="world">
-		<origin xyz="0.0 0.0 0.0"/>
-	</link>
-	<joint name="world_joint" type="fixed">
-		<parent link="world"/>
-		<child link="camera"/>
-		<origin rpy="0.0 0.0 0.0" xyz="0.0 0.0 0.0"/>
-	</joint>
-	<link name="camera">
-		<origin rpy="0.0 0.0 0.0" xyz="0.0 0.2 0.8"/>
-	</link>
-	<xacro:psm
-		prefix="one_"
-		parent_link="camera"
-		xyz="-0.25 0.0 0.5" rpy="0.0 0.0 3.1415926"
-		color="Green"
-	/>
-	<xacro:psm
-		prefix="two_"
-		parent_link="camera"
-		xyz="0.25 0.0 0.5" rpy="0.0 0.0 3.1415926"
-		color="Yellow"
-	/>
-	<!-- ros_control plugin -->
-	<gazebo>
-		<plugin name="gazebo_ros_control" filename="libgazebo_ros_control.so">
-			<robotNamespace>/davinci</robotNamespace>
-			<robotSimType>gazebo_ros_control/DefaultRobotHWSim</robotSimType>
-		</plugin>
-	</gazebo>
+    <xacro:include filename="$(find cwru_davinci_geometry_models)/model/psm.urdf.xacro"/>
+    <link name="world">
+        <origin xyz="0.0 0.0 0.0"/>
+    </link>
+    <joint name="world_joint" type="fixed">
+        <parent link="world"/>
+        <child link="camera"/>
+        <origin rpy="0.0 0.0 0.0" xyz="0.0 0.0 0.0"/>
+    </joint>
+    <link name="camera">
+        <origin rpy="0.0 0.0 0.0" xyz="0.0 0.2 0.8"/>
+    </link>
+    <xacro:psm_sca
+        prefix="one_"
+        parent_link="camera"
+        xyz="-0.25 0.0 0.5" rpy="0.0 0.0 3.1415926"
+        color="Green"/>
+    <xacro:psm_sca
+        prefix="two_"
+        parent_link="camera"
+        xyz="0.25 0.0 0.5" rpy="0.0 0.0 3.1415926"
+        color="Yellow"/>
+    <!-- ros_control plugin -->
+    <gazebo>
+        <plugin name="gazebo_ros_control" filename="libgazebo_ros_control.so">
+            <robotNamespace>/davinci</robotNamespace>
+            <robotSimType>gazebo_ros_control/DefaultRobotHWSim</robotSimType>
+        </plugin>
+    </gazebo>
 </robot>

File: model/psm.base.urdf.xacro (robot description, xacro)
@@ -29,5 +29,5 @@
 		</link>
 		<!-- joint 1 -->
-		<joint name="outer_yaw" type="revolute">
+		<joint name="${prefix}outer_yaw" type="revolute">
 			<parent link="${prefix}psm_base_link"/>
 			<child link="${prefix}outer_yaw_link"/>
@@ -59,5 +59,5 @@
 		<!-- link, all visual links mimic outer_pitch value -->
 		<!-- joint 2: outer_pitch -->
-		<joint name="outer_pitch" type="revolute">
+		<joint name="${prefix}outer_pitch" type="revolute">
 			<parent link="${prefix}outer_yaw_link"/>
 			<child link="${prefix}outer_pitch_link"/>
@@ -81,5 +81,5 @@
 		<!--wsn: for visualization links/joints of closed-chain mechanism, assign dynamic properties and control w/ fdbk-->
 		<!-- joint 2-1: outer_pitch_1 -->
-		<joint name="outer_pitch_1" type="continuous">
+		<joint name="${prefix}outer_pitch_1" type="continuous">
 			<parent link="${prefix}outer_yaw_link"/>
 			<child link="${prefix}outer_pitch_back_link"/>
@@ -88,5 +88,5 @@
 			<dynamics damping="1"/>
 			<origin rpy="-1.5708 -1.5708 0" xyz="0 0.0295 0.5185"/>
-			<mimic joint="outer_pitch" multiplier="1"/>
+			<mimic joint="${prefix}outer_pitch" multiplier="1"/>
 			<limit lower="-0.7854" upper="0.7854" velocity="5.0" effort="1000"/>
 		</joint>
@@ -110,10 +110,10 @@
 		</link>
 		<!-- joint 2-2: outer_pitch_2 -->
-		<joint name="outer_pitch_2" type="continuous">
+		<joint name="${prefix}outer_pitch_2" type="continuous">
 			<parent link="${prefix}outer_yaw_link"/>
 			<child link="${prefix}outer_pitch_front_link"/>
 			<axis xyz="0 0 1"/>
 			<origin rpy="-1.5708 -1.5708 0" xyz="0 0.0295 0.4285"/>
-			<mimic joint="outer_pitch" multiplier="1"/>
+			<mimic joint="${prefix}outer_pitch" multiplier="1"/>
 		</joint>
 		<!-- link 2-2: outer_pitch_front -->
@@ -136,10 +136,10 @@
 		</link>
 		<!-- joint 2-3: outer_pitch_3 -->
-		<joint name="outer_pitch_3" type="continuous">
+		<joint name="${prefix}outer_pitch_3" type="continuous">
 			<parent link="${prefix}outer_pitch_back_link"/>
 			<child link="${prefix}outer_pitch_bottom_link"/>
 			<axis xyz="0 0 1"/>
 			<origin rpy="0 0 0" xyz="0.04178 0.15007 -0.0137"/>
-			<mimic joint="outer_pitch" multiplier="-1"/>
+			<mimic joint="${prefix}outer_pitch" multiplier="-1"/>
 			<limit lower="-0.7854" upper="0.7854" velocity="5.0" effort="1000"/>
 			<dynamics damping="1"/>
@@ -164,10 +164,10 @@
 		</link>
 		<!-- joint 2-4: outer_pitch_4 -->
-		<joint name="outer_pitch_4" type="continuous">
+		<joint name="${prefix}outer_pitch_4" type="continuous">
 			<parent link="${prefix}outer_pitch_back_link"/>
 			<child link="${prefix}outer_pitch_top_link"/>
 			<axis xyz="0 0 1"/>
 			<origin rpy="0 0 0" xyz="0.04209 0.18695 -0.02412"/>
-			<mimic joint="outer_pitch" multiplier="-1"/>
+			<mimic joint="${prefix}outer_pitch" multiplier="-1"/>
 			<limit lower="-0.7854" upper="0.7854" velocity="5.0" effort="1000"/>
 			<dynamics damping="1"/>
@@ -192,10 +192,10 @@
 		</link>
 		<!-- joint 2-5: outer_pitch_5 -->
-		<joint name="outer_pitch_5" type="continuous">
+		<joint name="${prefix}outer_pitch_5" type="continuous">
 			<parent link="${prefix}outer_pitch_bottom_link"/>
 			<child link="${prefix}outer_insertion_link"/>
 			<axis xyz="0 0 1"/>
 			<origin rpy="0 0 0" xyz="-0.520 0 -0.0155"/>
-			<mimic joint="outer_pitch" multiplier="1"/>
+			<mimic joint="${prefix}outer_pitch" multiplier="1"/>
 			<limit lower="-0.7854" upper="0.7854" velocity="5.0" effort="1000"/>
 			<dynamics damping="1"/>
@@ -223,5 +223,5 @@
 		</gazebo>
 		<!-- joint 3: insertion -->
-		<joint name="outer_insertion" type="prismatic">
+		<joint name="${prefix}outer_insertion" type="prismatic">
 			<parent link="${prefix}outer_pitch_link"/>
 			<child link="${prefix}tool_main_link"/>
@@ -250,5 +250,5 @@
 		</link>
 		<!-- joint 4: Outer Roll -->
-		<joint name="outer_roll" type="revolute">
+		<joint name="${prefix}outer_roll" type="revolute">
 			<parent link="${prefix}tool_main_link"/>
 			<child link="${prefix}tool_wrist_link"/>
@@ -312,5 +312,5 @@
 		<transmission name="${prefix}tran2">
 			<type>transmission_interface/SimpleTransmission</type>
-			<joint name="outer_pitch">
+			<joint name="${prefix}outer_pitch">
 				<hardwareInterface>hardware_interface/EffortJointInterface</hardwareInterface>
 			</joint>
@@ -321,24 +321,24 @@
 		<gazebo>
 			<plugin name="mimic_1" filename="libroboticsgroup_gazebo_mimic_joint_plugin.so">
-				<joint>outer_pitch</joint>
-				<mimicJoint>outer_pitch_1</mimicJoint>
+				<joint>${prefix}outer_pitch</joint>
+				<mimicJoint>${prefix}outer_pitch_1</mimicJoint>
 			</plugin>
 			<plugin name="mimic_2" filename="libroboticsgroup_gazebo_mimic_joint_plugin.so">
-				<joint>outer_pitch</joint>
-				<mimicJoint>outer_pitch_2</mimicJoint>
+				<joint>${prefix}outer_pitch</joint>
+				<mimicJoint>${prefix}outer_pitch_2</mimicJoint>
 			</plugin>
 			<plugin name="mimic_3" filename="libroboticsgroup_gazebo_mimic_joint_plugin.so">
-				<joint>outer_pitch</joint>
-				<mimicJoint>outer_pitch_3</mimicJoint>
+				<joint>${prefix}outer_pitch</joint>
+				<mimicJoint>${prefix}outer_pitch_3</mimicJoint>
 				<multiplier>-1.0</multiplier>
 			</plugin>
 			<plugin name="mimic_4" filename="libroboticsgroup_gazebo_mimic_joint_plugin.so">
-				<joint>outer_pitch</joint>
-				<mimicJoint>outer_pitch_4</mimicJoint>
+				<joint>${prefix}outer_pitch</joint>
+				<mimicJoint>${prefix}outer_pitch_4</mimicJoint>
 				<multiplier>-1.0</multiplier>
 			</plugin>
 			<plugin name="mimic_5" filename="libroboticsgroup_gazebo_mimic_joint_plugin.so">
-				<joint>outer_pitch</joint>
-				<mimicJoint>outer_pitch_5</mimicJoint>
+				<joint>${prefix}outer_pitch</joint>
+				<mimicJoint>${prefix}outer_pitch_5</mimicJoint>
 			</plugin>
 		</gazebo>
@@ -354,5 +354,5 @@
 		<transmission name="${prefix}tran4">
 			<type>transmission_interface/SimpleTransmission</type>
-			<joint name="outer_roll">
+			<joint name="${prefix}outer_roll">
 				<hardwareInterface>hardware_interface/EffortJointInterface</hardwareInterface>
 			</joint>

File: model/psm.tool.sca.urdf.xacro (robot description, xacro)
@@ -2,9 +2,9 @@
 <robot name="dvrk_psm" xmlns:xacro="http://www.ros.org/wiki/xacro">
 	<!--This file contains different tool urdf -->
-	<xacro:include filename="$(find cwru_davinci_geometry_models)/model/common.urdf.xacro"/>
+	<!-- <xacro:include filename="$(find cwru_davinci_geometry_models)/model/common.urdf.xacro"/> -->
 	<!--sca-->
 	<xacro:macro name="psm_tool_sca" params="prefix">
 		<!-- joint 5: Outer wrist pitch joint -->
-		<joint name="outer_wrist_pitch" type="revolute">
+		<joint name="${prefix}outer_wrist_pitch" type="revolute">
 			<parent link="${prefix}tool_wrist_shaft_link"/>
 			<child link="${prefix}tool_wrist_sca_link"/>
@@ -36,8 +36,6 @@
 			</inertial>
 		</link>
-		<gazebo reference="${prefix}tool_wrist_sca_link">
-		</gazebo>
 		<!-- joint 6: Outer wrist yaw joint -->
-		<joint name="outer_wrist_yaw" type="revolute">
+		<joint name="${prefix}outer_wrist_yaw" type="revolute">
 			<parent link="${prefix}tool_wrist_sca_link"/>
 			<child link="${prefix}tool_wrist_sca_shaft_link"/>
@@ -62,5 +60,5 @@
 		</link>
 		<!-- joint 7-0: Outer open angle 1	-->
-		<joint name="jaw" type="revolute">
+		<joint name="${prefix}jaw" type="revolute">
 			<parent link="${prefix}tool_wrist_sca_shaft_link"/>
 			<child link="${prefix}tool_wrist_sca_ee_link_0"/>
@@ -84,5 +82,5 @@
 		</link>
 		<!-- joint 7-1: Outer open angle 1	-->
-		<joint name="jaw_mimic_1" type="revolute">
+		<joint name="${prefix}jaw_mimic_1" type="revolute">
 			<parent link="${prefix}tool_wrist_sca_shaft_link"/>
 			<child link="${prefix}tool_wrist_sca_ee_link_1"/>
@@ -90,5 +88,5 @@
 			<origin rpy="0 0 0" xyz="0 0 0"/>
 			<limit lower="-1.5707" upper="1.5707" velocity="10" effort="1000"/>
-			<mimic joint="jaw" multiplier="0.5"/>
+			<mimic joint="${prefix}jaw" multiplier="0.5"/>
 		</joint>
 		<!-- link 7-1: Outer open angle link 1 -->
@@ -107,5 +105,5 @@
 		</link>
 		<!-- joint 7-2: Outer open angle 2	 -->
-		<joint name="jaw_mimic_2" type="revolute">
+		<joint name="${prefix}jaw_mimic_2" type="revolute">
 			<parent link="${prefix}tool_wrist_sca_shaft_link"/>
 			<child link="${prefix}tool_wrist_sca_ee_link_2"/>
@@ -113,5 +111,5 @@
 			<origin rpy="0 0 0" xyz="0 0 0"/>
 			<limit lower="-1.5707" upper="1.5707" velocity="10" effort="1000"/>
-			<mimic joint="jaw" multiplier="-0.5"/>
+			<mimic joint="${prefix}jaw" multiplier="-0.5"/>
 		</joint>
 		<!-- link 7-2: Outer open angle link 2 -->
@@ -129,89 +127,4 @@
 			</inertial>
 		</link>
-		<link name="${prefix}fingertip2">
-			<visual>
-				<origin rpy="0 0 0" xyz="0.001 0.005 0.0005"/>
-				<geometry>
-					<box size="0.002 0.01 0.004"/>
-				</geometry>
-			</visual>
-			<collision>
-				<origin rpy="0 0 0" xyz="0.001 0.005 0.0005"/>
-				<geometry>
-					<box size="0.002 0.01 0.004"/>
-				</geometry>
-				<surface>
-					<friction>
-						<ode>
-							<mu>30.0</mu>
-							<mu2>30.0</mu2>
-						</ode>
-					</friction>
-					<contact>
-						<ode>
-							<kp>1000000.0</kp>
-							<kd>100.0</kd>
-							<max_vel>1.0</max_vel>
-							<min_depth>0.001</min_depth>
-						</ode>
-					</contact>
-				</surface>
-			</collision>
-			<inertial>
-				<origin xyz="0 0 0" rpy="0 0 0"/>
-				<mass value="0.05"/>
-				<inertia ixx="0.01" ixy="0.0" ixz="0.0" iyy="0.01" iyz="0.0" izz="0.005"/>
-			</inertial>
-		</link>
-		<!-- attach fingertip pad  -->
-		<joint name="${prefix}fingertip2_joint" type="fixed">
-			<parent link="${prefix}tool_wrist_sca_ee_link_2"/>
-			<child link="${prefix}fingertip2"/>
-			<axis xyz="0 0 1"/>
-			<origin rpy="0 0 0" xyz="0 0 0"/>
-		</joint>
-		<!-- wsn: other fingertip -->
-		<link name="${prefix}fingertip1">
-			<visual>
-				<origin rpy="0 0 0" xyz="-0.001 0.005 0.0005"/>
-				<geometry>
-					<box size="0.002 0.01 0.004"/>
-				</geometry>
-			</visual>
-			<collision name="${prefix}fingertip1_collision">
-				<origin rpy="0 0 0" xyz="-0.001 0.005 0.0005"/>
-				<geometry>
-					<box size="0.002 0.01 0.004"/>
-				</geometry>
-				<surface>
-					<friction>
-						<ode>
-							<mu>30.0</mu>
-							<mu2>30.0</mu2>
-						</ode>
-					</friction>
-					<contact>
-						<ode>
-							<kp>1000000.0</kp>
-							<kd>100.0</kd>
-							<max_vel>1.0</max_vel>
-							<min_depth>0.001</min_depth>
-						</ode>
-					</contact>
-				</surface>
-			</collision>
-			<inertial>
-				<origin xyz="0 0 0" rpy="0 0 0"/>
-				<mass value="0.05"/>
-				<inertia ixx="0.01" ixy="0.0" ixz="0.0" iyy="0.01" iyz="0.0" izz="0.005"/>
-			</inertial>
-		</link>
-		<!-- attach fingertip pad 1  -->
-		<joint name="${prefix}fingertip1_joint" type="fixed">
-			<parent link="${prefix}tool_wrist_sca_ee_link_1"/>
-			<child link="${prefix}fingertip1"/>
-			<axis xyz="0 0 1"/>
-			<origin rpy="0 0 0" xyz="0 0 0"/>
-		</joint>
 		<!-- tool tip -->
 		<!-- joint needs to be revolute (albeit immobile) to prevent Gazebo from optimizing the fiducial's position out.-->
@@ -219,5 +132,5 @@
 			<parent link="${prefix}tool_wrist_sca_shaft_link"/>
 			<child link="${prefix}tool_tip_link"/>
-			<origin rpy="0 ${PI/2} ${PI/2}" xyz="0 0.0102 0"/>
+			<origin rpy="0 ${pi/2} ${pi/2}" xyz="0 0.0102 0"/>
 		</joint>
 		<link name="${prefix}tool_tip_link">
@@ -227,4 +140,7 @@
 					<sphere radius="0.001"/>
 				</geometry>
+				<material name="green">
+						<color rgba="0 1.0 0 1.0"/>
+				</material>
 			</visual>
 			<!--Needs a dummy inertia value to link with the joint up above.-->
@@ -237,5 +153,7 @@
 		<!--this colors the tool-tip fiducial red; oddly, this shows up in the camera view, but NOT in the rviz view -->
 		<gazebo reference="${prefix}tool_tip_link">
-			<material>Gazebo/Red</material>
+			<material>Gazebo/Orange</material>
+		</gazebo>
+		<gazebo reference="${prefix}tool_wrist_sca_link">
 		</gazebo>
 		<!--Color the sticky fingertips pink, for visibility-->
@@ -244,13 +162,13 @@
 		</gazebo>
 		<!--Create the sticky fingertip.-->
-		<gazebo>
+<!-- 		<gazebo>
 			<plugin name="${prefix}fingertip1_finger" filename="libsticky_fingers.so">
 				<capacity>25</capacity>
 				<link>davinci_${prefix}::${prefix}tool_wrist_sca_ee_link_1</link>
 			</plugin>
-         	</gazebo>
+         	</gazebo> -->
 		<transmission name="${prefix}_tran5">
 			<type>transmission_interface/SimpleTransmission</type>
-			<joint name="outer_wrist_pitch">
+			<joint name="${prefix}outer_wrist_pitch">
 				<hardwareInterface>hardware_interface/EffortJointInterface</hardwareInterface>
 			</joint>
@@ -261,5 +179,5 @@
 		<transmission name="${prefix}_tran6">
 			<type>transmission_interface/SimpleTransmission</type>
-			<joint name="outer_wrist_yaw">
+			<joint name="${prefix}outer_wrist_yaw">
 				<hardwareInterface>hardware_interface/EffortJointInterface</hardwareInterface>
 			</joint>
@@ -270,5 +188,5 @@
 		<transmission name="${prefix}_tran7">
 			<type>transmission_interface/SimpleTransmission</type>
-			<joint name="jaw">
+			<joint name="${prefix}jaw">
 				<hardwareInterface>hardware_interface/EffortJointInterface</hardwareInterface>
 			</joint>
@@ -279,11 +197,11 @@
 		<gazebo>
 			<plugin name="mimic_6" filename="libroboticsgroup_gazebo_mimic_joint_plugin.so">
-				<joint>jaw</joint>
-				<mimicJoint>jaw_mimic_1</mimicJoint>
+				<joint>${prefix}jaw</joint>
+				<mimicJoint>${prefix}jaw_mimic_1</mimicJoint>
 				<multiplier>0.5</multiplier>
 			</plugin>
 			<plugin name="mimic_7" filename="libroboticsgroup_gazebo_mimic_joint_plugin.so">
-				<joint>jaw</joint>
-				<mimicJoint>jaw_mimic_2</mimicJoint>
+				<joint>${prefix}jaw</joint>
+				<mimicJoint>${prefix}jaw_mimic_2</mimicJoint>
 				<multiplier>-0.5</multiplier>
 			</plugin>

File: model/psm.urdf.xacro (robot description, xacro)
@@ -4,5 +4,5 @@
   <xacro:include filename="$(find cwru_davinci_geometry_models)/model/psm.base.urdf.xacro"/>
   <xacro:include filename="$(find cwru_davinci_geometry_models)/model/psm.tool.sca.urdf.xacro"/>
-  <xacro:include filename="$(find cwru_davinci_geometry_models)/model/psm.tool.caudier.urdf.xacro"/>
+  <!-- <xacro:include filename="$(find cwru_davinci_geometry_models)/model/psm.tool.caudier.urdf.xacro"/> -->
   <!-- Macro for psm with sca -->
   <xacro:macro name="psm_sca" params="prefix parent_link xyz rpy color">
@@ -15,6 +15,15 @@
         prefix="${prefix}"/>
   </xacro:macro>
+<!--   <xacro:macro name="psm_sca_two" params="prefix parent_link xyz rpy color">
+    <xacro:psm
+        prefix="${prefix}"
+        parent_link="${parent_link}"
+        xyz="${xyz}" rpy="${rpy}"
+        color="${color}"/>
+    <xacro:psm_tool_sca
+        prefix="${prefix}"/>
+  </xacro:macro> -->
   <!-- Macro for psm with caudier -->
-  <xacro:macro name="psm_caudier" params="prefix parent_link xyz rpy color">
+<!--   <xacro:macro name="psm_caudier" params="prefix parent_link xyz rpy color">
     <xacro:psm
         prefix="${prefix}"
@@ -24,4 +33,4 @@
     <xacro:psm_tool_caudier
         prefix="${prefix}"/>
-  </xacro:macro>
+  </xacro:macro> -->
 </robot>
