Commit message: Made modification in three .urdf.xacro files.
- Changed <robotNamespace> from 'davinci' to 'dvrk_psm' in file model/both_psms.urdf.xacro.

- Changed <hardwareInterface> from 'hardware_interface/EffortJointInterface' to 'hardware_interface/PositionJointInterface',
  Also removed '${prefix}' under mimic joint plugin in file model/psm.base.urdf.xacro.

- Changed <hardwareInterface> from 'hardware_interface/EffortJointInterface' to 'hardware_interface/PositionJointInterface',
  Also removed '${prefix}' under mimic joint plugin in file model/psm.tool.sca.urdf.xacro.

File: model/both_psms.urdf.xacro (robot description, xacro)
@@ -27,5 +27,5 @@
     <gazebo>
         <plugin name="gazebo_ros_control" filename="libgazebo_ros_control.so">
-            <robotNamespace>/davinci</robotNamespace>
+            <robotNamespace>/dvrk_psm</robotNamespace>
             <robotSimType>gazebo_ros_control/DefaultRobotHWSim</robotSimType>
         </plugin>

File: model/psm.base.urdf.xacro (robot description, xacro)
@@ -303,6 +303,6 @@
 		<transmission name="${prefix}tran1">
 			<type>transmission_interface/SimpleTransmission</type>
-			<joint name="outer_yaw">
-				<hardwareInterface>hardware_interface/EffortJointInterface</hardwareInterface>
+			<joint name="${prefix}outer_yaw">
+				<hardwareInterface>hardware_interface/PositionJointInterface</hardwareInterface>
 			</joint>
 			<actuator name="${prefix}motor1">
@@ -312,6 +312,6 @@
 		<transmission name="${prefix}tran2">
 			<type>transmission_interface/SimpleTransmission</type>
-			<joint name="${prefix}outer_pitch">
-				<hardwareInterface>hardware_interface/EffortJointInterface</hardwareInterface>
+			<joint name="outer_pitch">
+				<hardwareInterface>hardware_interface/PositionJointInterface</hardwareInterface>
 			</joint>
 			<actuator name="${prefix}motor2">
@@ -321,24 +321,24 @@
 		<gazebo>
 			<plugin name="mimic_1" filename="libroboticsgroup_gazebo_mimic_joint_plugin.so">
-				<joint>${prefix}outer_pitch</joint>
-				<mimicJoint>${prefix}outer_pitch_1</mimicJoint>
+				<joint>outer_pitch</joint>
+				<mimicJoint>outer_pitch_1</mimicJoint>
 			</plugin>
 			<plugin name="mimic_2" filename="libroboticsgroup_gazebo_mimic_joint_plugin.so">
-				<joint>${prefix}outer_pitch</joint>
-				<mimicJoint>${prefix}outer_pitch_2</mimicJoint>
+				<joint>outer_pitch</joint>
+				<mimicJoint>outer_pitch_2</mimicJoint>
 			</plugin>
 			<plugin name="mimic_3" filename="libroboticsgroup_gazebo_mimic_joint_plugin.so">
-				<joint>${prefix}outer_pitch</joint>
-				<mimicJoint>${prefix}outer_pitch_3</mimicJoint>
+				<joint>outer_pitch</joint>
+				<mimicJoint>outer_pitch_3</mimicJoint>
 				<multiplier>-1.0</multiplier>
 			</plugin>
 			<plugin name="mimic_4" filename="libroboticsgroup_gazebo_mimic_joint_plugin.so">
-				<joint>${prefix}outer_pitch</joint>
-				<mimicJoint>${prefix}outer_pitch_4</mimicJoint>
+				<joint>outer_pitch</joint>
+				<mimicJoint>outer_pitch_4</mimicJoint>
 				<multiplier>-1.0</multiplier>
 			</plugin>
 			<plugin name="mimic_5" filename="libroboticsgroup_gazebo_mimic_joint_plugin.so">
-				<joint>${prefix}outer_pitch</joint>
-				<mimicJoint>${prefix}outer_pitch_5</mimicJoint>
+				<joint>outer_pitch</joint>
+				<mimicJoint>outer_pitch_5</mimicJoint>
 			</plugin>
 		</gazebo>
@@ -346,5 +346,5 @@
 			<type>transmission_interface/SimpleTransmission</type>
 			<joint name="outer_insertion">
-				<hardwareInterface>hardware_interface/EffortJointInterface</hardwareInterface>
+				<hardwareInterface>hardware_interface/PositionJointInterface</hardwareInterface>
 			</joint>
 			<actuator name="${prefix}motor3">
@@ -354,6 +354,6 @@
 		<transmission name="${prefix}tran4">
 			<type>transmission_interface/SimpleTransmission</type>
-			<joint name="${prefix}outer_roll">
-				<hardwareInterface>hardware_interface/EffortJointInterface</hardwareInterface>
+			<joint name="outer_roll">
+				<hardwareInterface>hardware_interface/PositionJointInterface</hardwareInterface>
 			</joint>
 			<actuator name="${prefix}motor4">

File: model/psm.tool.sca.urdf.xacro (robot description, xacro)
@@ -170,6 +170,6 @@
 		<transmission name="${prefix}_tran5">
 			<type>transmission_interface/SimpleTransmission</type>
-			<joint name="${prefix}outer_wrist_pitch">
-				<hardwareInterface>hardware_interface/EffortJointInterface</hardwareInterface>
+			<joint name="outer_wrist_pitch">
+				<hardwareInterface>hardware_interface/PositionJointInterface</hardwareInterface>
 			</joint>
 			<actuator name="${prefix}_motor5">
@@ -179,6 +179,6 @@
 		<transmission name="${prefix}_tran6">
 			<type>transmission_interface/SimpleTransmission</type>
-			<joint name="${prefix}outer_wrist_yaw">
-				<hardwareInterface>hardware_interface/EffortJointInterface</hardwareInterface>
+			<joint name="outer_wrist_yaw">
+				<hardwareInterface>hardware_interface/PositionJointInterface</hardwareInterface>
 			</joint>
 			<actuator name="${prefix}_motor6">
@@ -188,6 +188,6 @@
 		<transmission name="${prefix}_tran7">
 			<type>transmission_interface/SimpleTransmission</type>
-			<joint name="${prefix}jaw">
-				<hardwareInterface>hardware_interface/EffortJointInterface</hardwareInterface>
+			<joint name="jaw">
+				<hardwareInterface>hardware_interface/PositionJointInterface</hardwareInterface>
 			</joint>
 			<actuator name="${prefix}_motor7">
@@ -197,11 +197,11 @@
 		<gazebo>
 			<plugin name="mimic_6" filename="libroboticsgroup_gazebo_mimic_joint_plugin.so">
-				<joint>${prefix}jaw</joint>
-				<mimicJoint>${prefix}jaw_mimic_1</mimicJoint>
+				<joint>jaw</joint>
+				<mimicJoint>jaw_mimic_1</mimicJoint>
 				<multiplier>0.5</multiplier>
 			</plugin>
 			<plugin name="mimic_7" filename="libroboticsgroup_gazebo_mimic_joint_plugin.so">
-				<joint>${prefix}jaw</joint>
-				<mimicJoint>${prefix}jaw_mimic_2</mimicJoint>
+				<joint>jaw</joint>
+				<mimicJoint>jaw_mimic_2</mimicJoint>
 				<multiplier>-0.5</multiplier>
 			</plugin>
