Commit message: Updated file psm and psm sca tool urdf file.

File: model/psm.base.urdf.xacro (robot description, xacro)
@@ -6,5 +6,5 @@
 	<xacro:macro name="psm" params="prefix parent_link xyz rpy color">
 		<!-- fixed joint -->
-		<joint name="${prefix}_fixed_joint" type="fixed">
+		<joint name="${prefix}fixed_joint" type="fixed">
 			<parent link="${parent_link}"/>
 			<child link="${prefix}psm_base_link"/>
@@ -312,5 +312,5 @@
 		<transmission name="${prefix}tran2">
 			<type>transmission_interface/SimpleTransmission</type>
-			<joint name="outer_pitch">
+			<joint name="${prefix}outer_pitch">
 				<hardwareInterface>hardware_interface/PositionJointInterface</hardwareInterface>
 			</joint>
@@ -321,29 +321,29 @@
 		<gazebo>
 			<plugin name="mimic_1" filename="libroboticsgroup_gazebo_mimic_joint_plugin.so">
-				<joint>outer_pitch</joint>
-				<mimicJoint>outer_pitch_1</mimicJoint>
+				<joint>${prefix}outer_pitch</joint>
+				<mimicJoint>${prefix}outer_pitch_1</mimicJoint>
 			</plugin>
 			<plugin name="mimic_2" filename="libroboticsgroup_gazebo_mimic_joint_plugin.so">
-				<joint>outer_pitch</joint>
-				<mimicJoint>outer_pitch_2</mimicJoint>
+				<joint>${prefix}outer_pitch</joint>
+				<mimicJoint>${prefix}outer_pitch_2</mimicJoint>
 			</plugin>
 			<plugin name="mimic_3" filename="libroboticsgroup_gazebo_mimic_joint_plugin.so">
-				<joint>outer_pitch</joint>
-				<mimicJoint>outer_pitch_3</mimicJoint>
+				<joint>${prefix}outer_pitch</joint>
+				<mimicJoint>${prefix}outer_pitch_3</mimicJoint>
 				<multiplier>-1.0</multiplier>
 			</plugin>
 			<plugin name="mimic_4" filename="libroboticsgroup_gazebo_mimic_joint_plugin.so">
-				<joint>outer_pitch</joint>
-				<mimicJoint>outer_pitch_4</mimicJoint>
+				<joint>${prefix}outer_pitch</joint>
+				<mimicJoint>${prefix}outer_pitch_4</mimicJoint>
 				<multiplier>-1.0</multiplier>
 			</plugin>
 			<plugin name="mimic_5" filename="libroboticsgroup_gazebo_mimic_joint_plugin.so">
-				<joint>outer_pitch</joint>
-				<mimicJoint>outer_pitch_5</mimicJoint>
+				<joint>${prefix}outer_pitch</joint>
+				<mimicJoint>${prefix}outer_pitch_5</mimicJoint>
 			</plugin>
 		</gazebo>
 		<transmission name="${prefix}tran3">
 			<type>transmission_interface/SimpleTransmission</type>
-			<joint name="outer_insertion">
+			<joint name="${prefix}outer_insertion">
 				<hardwareInterface>hardware_interface/PositionJointInterface</hardwareInterface>
 			</joint>
@@ -354,5 +354,5 @@
 		<transmission name="${prefix}tran4">
 			<type>transmission_interface/SimpleTransmission</type>
-			<joint name="outer_roll">
+			<joint name="${prefix}outer_roll">
 				<hardwareInterface>hardware_interface/PositionJointInterface</hardwareInterface>
 			</joint>

File: model/psm.tool.sca.urdf.xacro (robot description, xacro)
@@ -168,28 +168,28 @@
 			</plugin>
          	</gazebo> -->
-		<transmission name="${prefix}_tran5">
+		<transmission name="${prefix}tran5">
 			<type>transmission_interface/SimpleTransmission</type>
-			<joint name="outer_wrist_pitch">
+			<joint name="${prefix}outer_wrist_pitch">
 				<hardwareInterface>hardware_interface/PositionJointInterface</hardwareInterface>
 			</joint>
-			<actuator name="${prefix}_motor5">
+			<actuator name="${prefix}motor5">
 				<mechanicalReduction>1</mechanicalReduction>
 			</actuator>
 		</transmission>
-		<transmission name="${prefix}_tran6">
+		<transmission name="${prefix}tran6">
 			<type>transmission_interface/SimpleTransmission</type>
-			<joint name="outer_wrist_yaw">
+			<joint name="${prefix}outer_wrist_yaw">
 				<hardwareInterface>hardware_interface/PositionJointInterface</hardwareInterface>
 			</joint>
-			<actuator name="${prefix}_motor6">
+			<actuator name="${prefix}motor6">
 				<mechanicalReduction>1</mechanicalReduction>
 			</actuator>
 		</transmission>
-		<transmission name="${prefix}_tran7">
+		<transmission name="${prefix}tran7">
 			<type>transmission_interface/SimpleTransmission</type>
-			<joint name="jaw">
+			<joint name="${prefix}jaw">
 				<hardwareInterface>hardware_interface/PositionJointInterface</hardwareInterface>
 			</joint>
-			<actuator name="${prefix}_motor7">
+			<actuator name="${prefix}motor7">
 				<mechanicalReduction>1</mechanicalReduction>
 			</actuator>
@@ -197,11 +197,11 @@
 		<gazebo>
 			<plugin name="mimic_6" filename="libroboticsgroup_gazebo_mimic_joint_plugin.so">
-				<joint>jaw</joint>
-				<mimicJoint>jaw_mimic_1</mimicJoint>
+				<joint>${prefix}jaw</joint>
+				<mimicJoint>${prefix}jaw_mimic_1</mimicJoint>
 				<multiplier>0.5</multiplier>
 			</plugin>
 			<plugin name="mimic_7" filename="libroboticsgroup_gazebo_mimic_joint_plugin.so">
-				<joint>jaw</joint>
-				<mimicJoint>jaw_mimic_2</mimicJoint>
+				<joint>${prefix}jaw</joint>
+				<mimicJoint>${prefix}jaw_mimic_2</mimicJoint>
 				<multiplier>-0.5</multiplier>
 			</plugin>
