Commit message: Added two square bar model for testing needle collision detection in MoveIt! and made a modification.
- Added folder props/10mm_x_100mm_bar.

- Added folder props/5mm_x_100mm_bar.

- Modified model needle_r, corrected its collision model.

File: model/psm.tool.sca.urdf.xacro (robot description, xacro)
@@ -127,4 +127,95 @@
 			</inertial>
 		</link>
+		<link name="${prefix}fingertip2">
+			<visual>
+				<origin rpy="0 0 0" xyz="0.001 0.005 0.0005"/>
+				<geometry>
+					<box size="0.002 0.01 0.004"/>
+				</geometry>
+				<material name="green">
+						<color rgba="0 1.0 0 1.0"/>
+				</material>
+			</visual>
+			<collision>
+				<origin rpy="0 0 0" xyz="0.001 0.005 0.0005"/>
+				<geometry>
+					<box size="0.002 0.01 0.004"/>
+				</geometry>
+				<surface>
+					<friction>
+						<ode>
+							<mu>30.0</mu>
+							<mu2>30.0</mu2>
+						</ode>
+					</friction>
+					<contact>
+						<ode>
+							<kp>1000000.0</kp>
+							<kd>100.0</kd>
+							<max_vel>1.0</max_vel>
+							<min_depth>0.001</min_depth>
+						</ode>
+					</contact>
+				</surface>
+			</collision>
+			<inertial>
+				<origin xyz="0 0 0" rpy="0 0 0"/>
+				<mass value="0.05"/>
+				<inertia ixx="0.01" ixy="0.0" ixz="0.0" iyy="0.01" iyz="0.0" izz="0.005"/>
+			</inertial>
+		</link>
+		<!-- attach fingertip pad  -->
+		<joint name="${prefix}fingertip2_joint" type="fixed">
+			<parent link="${prefix}tool_wrist_sca_ee_link_2"/>
+			<child link="${prefix}fingertip2"/>
+			<axis xyz="0 0 1"/>
+			<origin rpy="0 0 0" xyz="0 0 0"/>
+		</joint>
+		<!-- wsn: other fingertip -->
+		<link name="${prefix}fingertip1">
+			<visual>
+				<origin rpy="0 0 0" xyz="-0.001 0.005 0.0005"/>
+				<geometry>
+					<box size="0.002 0.01 0.004"/>
+				</geometry>
+				<material name="green">
+						<color rgba="0 1.0 0 1.0"/>
+				</material>
+			</visual>
+			<collision name="${prefix}fingertip1_collision">
+				<origin rpy="0 0 0" xyz="-0.001 0.005 0.0005"/>
+				<geometry>
+					<box size="0.002 0.01 0.004"/>
+				</geometry>
+				<surface>
+					<friction>
+						<ode>
+							<mu>30.0</mu>
+							<mu2>30.0</mu2>
+						</ode>
+					</friction>
+					<contact>
+						<ode>
+							<kp>1000000.0</kp>
+							<kd>100.0</kd>
+							<max_vel>1.0</max_vel>
+							<min_depth>0.001</min_depth>
+						</ode>
+					</contact>
+				</surface>
+			</collision>
+			<inertial>
+				<origin xyz="0 0 0" rpy="0 0 0"/>
+				<mass value="0.05"/>
+				<inertia ixx="0.01" ixy="0.0" ixz="0.0" iyy="0.01" iyz="0.0" izz="0.005"/>
+			</inertial>
+		</link>
+		<!-- attach fingertip pad 1  -->
+		<joint name="${prefix}fingertip1_joint" type="fixed">
+			<parent link="${prefix}tool_wrist_sca_ee_link_1"/>
+			<child link="${prefix}fingertip1"/>
+			<axis xyz="0 0 1"/>
+			<origin rpy="0 0 0" xyz="0 0 0"/>
+		</joint>
 		<!-- tool tip -->
 		<!-- joint needs to be revolute (albeit immobile) to prevent Gazebo from optimizing the fiducial's position out.-->
@@ -162,10 +253,11 @@
 		</gazebo>
 		<!--Create the sticky fingertip.-->
-<!-- 		<gazebo>
+		<gazebo>
 			<plugin name="${prefix}fingertip1_finger" filename="libsticky_fingers.so">
 				<capacity>25</capacity>
-				<link>davinci_${prefix}::${prefix}tool_wrist_sca_ee_link_1</link>
+				<!-- <link>davinci_${prefix}::${prefix}tool_wrist_sca_ee_link_1</link> -->
+				<link>dvrk_psm::${prefix}tool_wrist_sca_ee_link_1</link>
 			</plugin>
-         	</gazebo> -->
+		</gazebo>
 		<transmission name="${prefix}tran5">
 			<type>transmission_interface/SimpleTransmission</type>
