Commit message: HW-MoveIt integration.

File: model_with_prefix/PSM1.urdf.xacro (robot description, xacro)
@@ -2,5 +2,5 @@
 <robot name="dvrk_psm" xmlns:xacro="http://www.ros.org/wiki/xacro">
   <!-- Macros -->
-  <xacro:include filename="$(find cwru_davinci_geometry_models)/model/psm.urdf.xacro"/>
+  <xacro:include filename="$(find cwru_davinci_geometry_models)/model_with_prefix/psm.urdf.xacro"/>
   <link name="world"/>
   <xacro:psm_sca

File: model_with_prefix/PSM2.urdf.xacro (robot description, xacro)
@@ -5,5 +5,5 @@
   <link name="world"/>
   <xacro:psm_sca
-      prefix="PSM2/"
+      prefix="PSM2"
       parent_link="world"
       xyz="0.25 0.0 0.5" rpy="0.0 0.0 -3.1415926"

File: model_with_prefix/both_psms.urdf.xacro (robot description, xacro)
@@ -2,5 +2,5 @@
 <robot name="dvrk_psm" xmlns:xacro="http://www.ros.org/wiki/xacro">
 <!-- Macros -->
-    <xacro:include filename="$(find cwru_davinci_geometry_models)/model/psm.urdf.xacro"/>
+    <xacro:include filename="$(find cwru_davinci_geometry_models)/model_with_prefix/psm.urdf.xacro"/>
     <link name="world">
         <origin xyz="0.0 0.0 0.0"/>

File: model_with_prefix/psm.tool.sca.urdf.xacro (robot description, xacro)
@@ -2,9 +2,9 @@
 <robot name="dvrk_psm" xmlns:xacro="http://www.ros.org/wiki/xacro">
 	<!--This file contains different tool urdf -->
-	<xacro:include filename="$(find cwru_davinci_geometry_models)/model/common.urdf.xacro"/>
+	<xacro:include filename="$(find cwru_davinci_geometry_models)/model_with_prefix/common.urdf.xacro"/>
 	<!--sca-->
 	<xacro:macro name="psm_tool_sca" params="prefix">
 		<!-- joint 5: Outer wrist pitch joint -->
-		<joint name="outer_wrist_pitch" type="revolute">
+		<joint name="${prefix}outer_wrist_pitch" type="revolute">
 			<parent link="${prefix}tool_wrist_shaft_link"/>
 			<child link="${prefix}tool_wrist_sca_link"/>
@@ -37,5 +37,5 @@
 		</link>
 		<!-- joint 6: Outer wrist yaw joint -->
-		<joint name="outer_wrist_yaw" type="revolute">
+		<joint name="${prefix}outer_wrist_yaw" type="revolute">
 			<parent link="${prefix}tool_wrist_sca_link"/>
 			<child link="${prefix}tool_wrist_sca_shaft_link"/>
@@ -60,5 +60,5 @@
 		</link>
 		<!-- joint 7-0: Outer open angle 1	-->
-		<joint name="jaw" type="revolute">
+		<joint name="${prefix}jaw" type="revolute">
 			<parent link="${prefix}tool_wrist_sca_shaft_link"/>
 			<child link="${prefix}tool_wrist_sca_ee_link_0"/>
@@ -82,5 +82,5 @@
 		</link>
 		<!-- joint 7-1: Outer open angle 1	-->
-		<joint name="jaw_mimic_1" type="revolute">
+		<joint name="${prefix}jaw_mimic_1" type="revolute">
 			<parent link="${prefix}tool_wrist_sca_shaft_link"/>
 			<child link="${prefix}tool_wrist_sca_ee_link_1"/>
@@ -88,5 +88,5 @@
 			<origin rpy="0 0 0" xyz="0 0 0"/>
 			<limit lower="-1.5707" upper="1.5707" velocity="10" effort="1000"/>
-			<mimic joint="jaw" multiplier="0.5"/>
+			<mimic joint="${prefix}jaw" multiplier="0.5"/>
 		</joint>
 		<!-- link 7-1: Outer open angle link 1 -->
@@ -105,5 +105,5 @@
 		</link>
 		<!-- joint 7-2: Outer open angle 2	 -->
-		<joint name="jaw_mimic_2" type="revolute">
+		<joint name="${prefix}jaw_mimic_2" type="revolute">
 			<parent link="${prefix}tool_wrist_sca_shaft_link"/>
 			<child link="${prefix}tool_wrist_sca_ee_link_2"/>
@@ -111,5 +111,5 @@
 			<origin rpy="0 0 0" xyz="0 0 0"/>
 			<limit lower="-1.5707" upper="1.5707" velocity="10" effort="1000"/>
-			<mimic joint="jaw" multiplier="-0.5"/>
+			<mimic joint="${prefix}jaw" multiplier="-0.5"/>
 		</joint>
 		<!-- link 7-2: Outer open angle link 2 -->
@@ -262,6 +262,6 @@
 		<transmission name="${prefix}tran5">
 			<type>transmission_interface/SimpleTransmission</type>
-			<joint name="outer_wrist_pitch">
-				<hardwareInterface>hardware_interface/EffortJointInterface</hardwareInterface>
+			<joint name="${prefix}outer_wrist_pitch">
+				<hardwareInterface>hardware_interface/PositionJointInterface</hardwareInterface>
 			</joint>
 			<actuator name="${prefix}motor5">
@@ -271,6 +271,6 @@
 		<transmission name="${prefix}tran6">
 			<type>transmission_interface/SimpleTransmission</type>
-			<joint name="outer_wrist_yaw">
-				<hardwareInterface>hardware_interface/EffortJointInterface</hardwareInterface>
+			<joint name="${prefix}outer_wrist_yaw">
+				<hardwareInterface>hardware_interface/PositionJointInterface</hardwareInterface>
 			</joint>
 			<actuator name="${prefix}motor6">
@@ -280,6 +280,6 @@
 		<transmission name="${prefix}tran7">
 			<type>transmission_interface/SimpleTransmission</type>
-			<joint name="jaw">
-				<hardwareInterface>hardware_interface/EffortJointInterface</hardwareInterface>
+			<joint name="${prefix}jaw">
+				<hardwareInterface>hardware_interface/PositionJointInterface</hardwareInterface>
 			</joint>
 			<actuator name="${prefix}motor7">
@@ -289,11 +289,11 @@
 		<gazebo>
 			<plugin name="mimic_6" filename="libroboticsgroup_gazebo_mimic_joint_plugin.so">
-				<joint>jaw</joint>
-				<mimicJoint>jaw_mimic_1</mimicJoint>
+				<joint>${prefix}jaw</joint>
+				<mimicJoint>${prefix}jaw_mimic_1</mimicJoint>
 				<multiplier>0.5</multiplier>
 			</plugin>
 			<plugin name="mimic_7" filename="libroboticsgroup_gazebo_mimic_joint_plugin.so">
-				<joint>jaw</joint>
-				<mimicJoint>jaw_mimic_2</mimicJoint>
+				<joint>${prefix}jaw</joint>
+				<mimicJoint>${prefix}jaw_mimic_2</mimicJoint>
 				<multiplier>-0.5</multiplier>
 			</plugin>

File: model_with_prefix/psm.urdf.xacro (robot description, xacro)
@@ -2,6 +2,6 @@
 <robot name="dvrk_psm" xmlns:xacro="http://www.ros.org/wiki/xacro">
   <!-- Macros -->
-  <xacro:include filename="$(find cwru_davinci_geometry_models)/model/psm.base.urdf.xacro"/>
-  <xacro:include filename="$(find cwru_davinci_geometry_models)/model/psm.tool.sca.urdf.xacro"/>
+  <xacro:include filename="$(find cwru_davinci_geometry_models)/model_with_prefix/psm.base.urdf.xacro"/>
+  <xacro:include filename="$(find cwru_davinci_geometry_models)/model_with_prefix/psm.tool.sca.urdf.xacro"/>
   <!-- <xacro:include filename="$(find cwru_davinci_geometry_models)/model/psm.tool.caudier.urdf.xacro"/> -->
   <!-- Macro for psm with sca -->
